File: SteeringServo/SteeringServo.kicad_pcb (KiCad board)
At the start: 2 copper layers, 78.1 x 47 mm, 12 parts, among them J1 MotorConnector, J2 To 12V Converter, J3 Signal, J4 Signal, SW1 SW_Push, U1 TLE5205, U2 StatusLED, U3 L7805

Commit message: new routing
Parts:
- added R1: R10k, Resistor_THT:R_Axial_DIN0309_L9.0mm_D3.2mm_P5.08mm_Vertical, F.Cu at (218.4, 59.7)
Routing:
- net 5V: track 92.8 -> 98.6 mm
- net M_IN_1: track 48.2 -> 52.9 mm
- net GND: track 213.7 -> 216.6 mm
Changed lines of the file:
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@@
-(kicad_pcb (version 20171130) (host pcbnew "(5.0.0)")
+(kicad_pcb (version 20171130) (host pcbnew 5.1.0)
   (general
     (thickness 1.6)
     (drawings 4)
-    (tracks 206)
+    (tracks 215)
     (zones 0)
-    (modules 12)
+    (modules 13)
     (nets 38)
   )
@@
   )
   (setup
-    (last_trace_width 2)
+    (last_trace_width 1.5)
     (user_trace_width 1)
     (user_trace_width 1.5)
@@
     (zone_45_only no)
     (trace_min 0.2)
-    (segment_width 0.2)
-    (edge_width 0.1)
     (via_size 0.8)
     (via_drill 0.4)
@@
     (uvia_min_size 0.2)
     (uvia_min_drill 0.1)
+    (edge_width 0.1)
+    (segment_width 0.2)
     (pcb_text_width 0.3)
     (pcb_text_size 1.5 1.5)
@@
     (add_net SERVO_POTI)
     (add_net Signal)
+  )
+  (module Resistor_THT:R_Axial_DIN0309_L9.0mm_D3.2mm_P5.08mm_Vertical (layer F.Cu)
+    (at 218.44 59.69 270)
+    (descr "Resistor, Axial_DIN0309 series, Axial, Vertical, pin pitch=5.08mm, 0.5W = 1/2W, length*diameter=9*3.2mm^2, http://cdn-reichelt.de/documents/datenblatt/B400/1_4W%23YAG.pdf")
+    (tags "Resistor Axial_DIN0309 series Axial Vertical pin pitch 5.08mm 0.5W = 1/2W length 9mm diameter 3.2mm")
+    (fp_text reference R1 (at 2.54 -2.72 270) (layer F.SilkS)
+      (effects (font (size 1 1) (thickness 0.15)))
+    )
+    (fp_text value R10k (at 2.54 2.72 270) (layer F.Fab)
+      (effects (font (size 1 1) (thickness 0.15)))
+    )
+    (fp_text user %R (at 2.54 -2.72 270) (layer F.Fab)
+      (effects (font (size 1 1) (thickness 0.15)))
+    )
+    (fp_line (start 6.13 -1.85) (end -1.85 -1.85) (layer F.CrtYd) (width 0.05))
+    (fp_line (start 6.13 1.85) (end 6.13 -1.85) (layer F.CrtYd) (width 0.05))
+    (fp_line (start -1.85 1.85) (end 6.13 1.85) (layer F.CrtYd) (width 0.05))
+    (fp_line (start -1.85 -1.85) (end -1.85 1.85) (layer F.CrtYd) (width 0.05))
+    (fp_line (start 1.72 0) (end 3.98 0) (layer F.SilkS) (width 0.12))
+    (fp_line (start 0 0) (end 5.08 0) (layer F.Fab) (width 0.1))
+    (fp_circle (center 0 0) (end 1.72 0) (layer F.SilkS) (width 0.12))
+    (fp_circle (center 0 0) (end 1.6 0) (layer F.Fab) (width 0.1))
+    (pad 2 thru_hole oval (at 5.08 0 270) (size 1.6 1.6) (drill 0.8) (layers *.Cu *.Mask)
+      (net 3 5V))
+    (pad 1 thru_hole circle (at 0 0 270) (size 1.6 1.6) (drill 0.8) (layers *.Cu *.Mask)
+      (net 15 M_IN_1))
+    (model ${KISYS3DMOD}/Resistor_THT.3dshapes/R_Axial_DIN0309_L9.0mm_D3.2mm_P5.08mm_Vertical.wrl
+      (at (xyz 0 0 0))
+      (scale (xyz 1 1 1))
+      (rotate (xyz 0 0 0))
+    )
   )
   (module Package_TO_SOT_THT:TO-220-3_Vertical (layer F.Cu)
@@
   (segment (start 202.565 37.465) (end 200.025 34.925) (width 2) (layer B.Cu) (net 3))
   (segment (start 202.565 40.005) (end 202.565 37.465) (width 2) (layer B.Cu) (net 3))
+  (segment (start 216.535 66.675) (end 213.480002 66.675) (width 2) (layer B.Cu) (net 3))
+  (segment (start 218.44 64.77) (end 216.535 66.675) (width 2) (layer B.Cu) (net 3))
   (segment (start 175.955 46.99) (end 166.805 46.99) (width 1) (layer B.Cu) (net 4))
   (segment (start 170.18 68.205) (end 169.17 69.215) (width 1) (layer B.Cu) (net 4))
@@
   (segment (start 161.105 67.76) (end 161.105 52.69) (width 1.5) (layer B.Cu) (net 4))
   (segment (start 214.08001 59.54) (end 213.79001 59.83) (width 1.5) (layer B.Cu) (net 4))
-  (segment (start 228.6 59.54) (end 214.08001 59.54) (width 1.5) (layer B.Cu) (net 4))
   (segment (start 197.485 34.925) (end 197.485 40.005) (width 2) (layer B.Cu) (net 4))
   (segment (start 178.29637 30.56) (end 177.165 30.56) (width 2) (layer B.Cu) (net 4))
@@
   (segment (start 196.35 30.79) (end 207.645 30.79) (width 2) (layer B.Cu) (net 4))
   (segment (start 196.12 30.56) (end 196.35 30.79) (width 2) (layer B.Cu) (net 4))
+  (segment (start 215.53227 59.54) (end 215.68227 59.69) (width 1.5) (layer B.Cu) (net 4))
+  (segment (start 214.08001 59.54) (end 215.53227 59.54) (width 1.5) (layer B.Cu) (net 4))
+  (segment (start 215.68227 59.69) (end 215.68227 60.74227) (width 1.5) (layer B.Cu) (net 4))
+  (segment (start 215.68227 60.74227) (end 217.17 62.23) (width 1.5) (layer B.Cu) (net 4))
+  (segment (start 225.91 62.23) (end 228.6 59.54) (width 1.5) (layer B.Cu) (net 4))
+  (segment (start 217.17 62.23) (end 225.91 62.23) (width 1.5) (layer B.Cu) (net 4))
   (segment (start 175.955 43.18) (end 175.955 41.335) (width 1) (layer B.Cu) (net 5))
   (segment (start 175.955 41.335) (end 177.92 39.37) (width 3) (layer B.Cu) (net 5))
@@
   (segment (start 179.255 45.72) (end 179.80998 46.27498) (width 1) (layer B.Cu) (net 15))
   (segment (start 175.955 45.72) (end 179.255 45.72) (width 1) (layer B.Cu) (net 15))
+  (segment (start 217.805 59.055) (end 218.44 59.69) (width 2) (layer B.Cu) (net 15))
+  (segment (start 217.805 55.245) (end 217.805 59.055) (width 2) (layer B.Cu) (net 15))
   (segment (start 222.885 55.245) (end 222.885 56.515) (width 2) (layer B.Cu) (net 16))
   (segment (start 222.885 55.245) (end 222.885 53.975) (width 2) (layer B.Cu) (net 16))
